Commit message: Added a virtual link in the xacro description to allow better cloud visualization with rviz

File: urdf/ensenso_n35.urdf.xacro (robot description, xacro)
@@ -90,4 +90,18 @@
             </collision>
         </link>
+        <!-- Virtual cloud -->
+        <joint name="${name}_virtual_cloud_joint" type="fixed">
+            <parent link="${name}_body"/>
+            <child link="${name}_virtual_cloud"/>
+            <origin xyz="0.0 0.0 1.5" rpy="3.141592 0.0 0.0"/>
+        </joint>
+        <link name="${name}_virtual_cloud">
+            <visual>
+                <origin xyz="0 0 0" rpy="0 0 0"/>
+                <geometry>
+                    <cylinder length="0.001" radius="0.022"/>
+                </geometry>
+            </visual>
+        </link>
     </xacro:macro>
 </robot>

Commit message: Removes geometry from virtual cloud link
/cc @andreucm

File: urdf/ensenso_n35.urdf.xacro (robot description, xacro)
@@ -96,12 +96,5 @@
             <origin xyz="0.0 0.0 1.5" rpy="3.141592 0.0 0.0"/>
         </joint>
-        <link name="${name}_virtual_cloud">
-            <visual>
-                <origin xyz="0 0 0" rpy="0 0 0"/>
-                <geometry>
-                    <cylinder length="0.001" radius="0.022"/>
-                </geometry>
-            </visual>
-        </link>
+        <link name="${name}_virtual_cloud" />
     </xacro:macro>
 </robot>

Commit message: Adds: * Param focus length.. the distance to the middle of the box where the precision is good, this place a frame at this distance * gazebo_ros_openni_kinect plugin to simulate the ensenso, most of the parameters are tuned for the N35. The parameter focus length also defines the point cloud cut off limits of the plugin

File: urdf/ensenso_n35.urdf.xacro (robot description, xacro)
@@ -1,100 +1,146 @@
 <?xml version="1.0"?>
-<robot xmlns:xacro="http://ros.org/wiki/xacro"
-       name="ensenso_nx">
-    <!-- Colors -->
-    <material name="Ensenso/Blue">
-        <color rgba="0.1 0.1 1.0 1.0"/>
-    </material>
-    <material name="Ensenso/Grey">
-        <color rgba="0.4 0.4 0.4 1.0"/>
-    </material>
-    <material name="Ensenso/Black">
-        <color rgba="0.05 0.05 0.05 1.0"/>
-    </material>
-    <material name="Ensenso/White">
-        <color rgba="0.9 0.9 0.9 0.6"/>
-    </material>
-    <xacro:macro name="ensenso_n35" params="name parent *origin">
-        <!-- The Ensenso N35 camera -->
-        <joint name="${parent}_${name}_joint" type="fixed">
-            <xacro:insert_block name="origin"/>
-            <parent link="${parent}" />
-            <child link="${name}_body" />
-        </joint>
-        <link name="${name}_body">
-            <visual>
-                <origin xyz="0.0875 -0.025 -0.026" rpy="0 0 0"/>
-                <geometry>
-                    <mesh filename="package://ensenso_nx/urdf/meshes/N30-602-16.stl" scale="0.001 0.001 0.001"/>
-                </geometry>
-                <material name="Ensenso/Blue"/>
-            </visual>
-            <collision>
-                <origin xyz="0.01 0 0.01" rpy="0 0 0"/>
-                <geometry>
-                    <!-- box size="0.175 0.050 0.052"/ -->
-                    <box size="0.220 0.1 0.1"/>
-                </geometry>
-            </collision>
-        </link>
-        <!-- Useful reference frames -->
-        <!-- Lens left -->
-        <joint name="${name}_lens_left_joint" type="fixed">
-            <parent link="${name}_body"/>
-            <child link="${name}_lens_left"/>
-            <origin xyz="-0.05 0.0 0.026" rpy="0.0 0.0 0.0"/>
-        </joint>
-        <link name="${name}_lens_left">
-            <visual>
-                <origin xyz="0 0 0" rpy="0 0 0"/>
-                <geometry>
-                    <cylinder length="0.001" radius="0.015"/>
-                </geometry>
-                <material name="Ensenso/White"/>
-            </visual>
-        </link>
-        <!-- Lens right -->
-        <joint name="${name}_lens_right_joint" type="fixed">
-            <parent link="${name}_body"/>
-            <child link="${name}_lens_right"/>
-            <origin xyz="0.05 0.0 0.026" rpy="0.0 0.0 0.0"/>
-        </joint>
-        <link name="${name}_lens_right">
-            <visual>
-                <origin xyz="0 0 0" rpy="0 0 0"/>
-                <geometry>
-                    <cylinder length="0.001" radius="0.015"/>
-                </geometry>
-                <material name="Ensenso/White"/>
-            </visual>
-        </link>
-        <!-- Emitter -->
-        <joint name="${name}_emitter_joint" type="fixed">
-            <parent link="${name}_body"/>
-            <child link="${name}_emitter"/>
-            <origin xyz="0.0 0.0 0.026" rpy="0.0 0.0 0.0"/>
-        </joint>
-        <link name="${name}_emitter">
-            <visual>
-                <origin xyz="0 0 0" rpy="0 0 0"/>
-                <geometry>
-                    <cylinder length="0.001" radius="0.022"/>
-                </geometry>
-                <material name="Ensenso/White"/>
-            </visual>
-            <collision>
-                <origin xyz="0 0 0" rpy="0 0 0"/>
-                <geometry>
-                    <cylinder length="0.001" radius="0.015"/>
-                </geometry>
-            </collision>
-        </link>
-        <!-- Virtual cloud -->
-        <joint name="${name}_virtual_cloud_joint" type="fixed">
-            <parent link="${name}_body"/>
-            <child link="${name}_virtual_cloud"/>
-            <origin xyz="0.0 0.0 1.5" rpy="3.141592 0.0 0.0"/>
-        </joint>
-        <link name="${name}_virtual_cloud" />
-    </xacro:macro>
+<robot xmlns:xacro="http://ros.org/wiki/xacro" name="ensenso_nx">
+<!-- Colors -->
+<material name="Ensenso/Blue">
+	<color rgba="0.1 0.1 1.0 1.0"/>
+</material>
+<material name="Ensenso/Grey">
+	<color rgba="0.4 0.4 0.4 1.0"/>
+</material>
+<material name="Ensenso/Black">
+	<color rgba="0.05 0.05 0.05 1.0"/>
+</material>
+<material name="Ensenso/White">
+	<color rgba="0.9 0.9 0.9 0.6"/>
+</material>
+<xacro:macro name="ensenso_n35" params="name parent focus_length=1.5 *origin">
+	<!-- The Ensenso N35 camera -->
+	<joint name="${parent}_${name}_joint" type="fixed">
+		<xacro:insert_block name="origin"/>
+		<parent link="${parent}" />
+		<child link="${name}_body" />
+	</joint>
+	<link name="${name}_body">
+		<visual>
+			<origin xyz="0.0875 -0.025 -0.026" rpy="0 0 0"/>
+			<geometry>
+				<mesh filename="package://ensenso_nx/urdf/meshes/N30-602-16.stl" scale="0.001 0.001 0.001"/>
+			</geometry>
+			<material name="Ensenso/Blue"/>
+		</visual>
+		<collision>
+			<origin xyz="0.01 0 0.01" rpy="0 0 0"/>
+			<geometry>
+				<box size="0.220 0.1 0.1"/>
+			</geometry>
+		</collision>
+		<inertial>
+			<mass value="0.5" />
+			<origin xyz="0 0 0" rpy="0 0 0"/>
+			<inertia ixx="${0.0833333 * 0.5 * (0.1*0.1 + 0.1*0.1)}" ixy="0.0" ixz="0.0"
+			iyy="${0.0833333 * 0.5 * (0.220*0.220 + 0.1*0.1)}" iyz="0.0"
+			izz="${0.0833333 * 0.5 * (0.220*0.220 + 0.1*0.1)}" />
+		</inertial>
+	</link>
+	<!-- Useful reference frames -->
+	<!-- Lens left -->
+	<joint name="${name}_lens_left_joint" type="fixed">
+		<parent link="${name}_body"/>
+		<child link="${name}_lens_left"/>
+		<origin xyz="-0.05 0.0 0.026" rpy="0.0 0.0 0.0"/>
+	</joint>
+	<link name="${name}_lens_left">
+		<visual>
+			<origin xyz="0 0 0" rpy="0 0 0"/>
+			<geometry>
+				<cylinder length="0.001" radius="0.015"/>
+			</geometry>
+			<material name="Ensenso/White"/>
+		</visual>
+	</link>
+	<!-- Lens right -->
+	<joint name="${name}_lens_right_joint" type="fixed">
+		<parent link="${name}_body"/>
+		<child link="${name}_lens_right"/>
+		<origin xyz="0.05 0.0 0.026" rpy="0.0 0.0 0.0"/>
+	</joint>
+	<link name="${name}_lens_right">
+		<visual>
+			<origin xyz="0 0 0" rpy="0 0 0"/>
+			<geometry>
+				<cylinder length="0.001" radius="0.015"/>
+			</geometry>
+			<material name="Ensenso/White"/>
+		</visual>
+	</link>
+	<!-- Emitter -->
+	<joint name="${name}_emitter_joint" type="fixed">
+		<parent link="${name}_body"/>
+		<child link="${name}_emitter"/>
+		<origin xyz="0.0 0.0 0.026" rpy="0.0 0.0 0.0"/>
+	</joint>
+	<link name="${name}_emitter">
+		<visual>
+			<origin xyz="0 0 0" rpy="0 0 0"/>
+			<geometry>
+				<cylinder length="0.001" radius="0.022"/>
+			</geometry>
+			<material name="Ensenso/White"/>
+		</visual>
+		<collision>
+			<origin xyz="0 0 0" rpy="0 0 0"/>
+			<geometry>
+				<cylinder length="0.001" radius="0.015"/>
+			</geometry>
+		</collision>
+	</link>
+	<!-- Focus point for several models of N35 -->
+	<joint name="${name}_focus_joint" type="fixed">
+		<parent link="${name}_body"/>
+		<child link="${name}_focus_cloud"/>
+		<origin xyz="0.0 0.0 ${focus_length}" rpy="3.141592 0.0 0.0"/>
+	</joint>
+	<link name="${name}_focus_cloud" />
+	<gazebo reference="${name}_body">
+		<sensor name="ensenso_camera" type="depth">
+			<!-- openni plugin has the x pointing towards the scene, so rotate to have z -->
+			<pose frame="${name}_body">0.0 0.0 0.0 0.0 -1.5708 0.0</pose>
+			<camera>
+				<horizontal_fov>0.74839718</horizontal_fov>
+				<image>
+					<width>1280</width>
+					<height>1024</height>
+					<format>R8G8B8</format>
+				</image>
+				<clip>
+					<near>0.1</near>
+					<far>10.0</far>
+				</clip>
+				<noise>
+					<type>gaussian</type>
+					<mean>0.5</mean>
+					<stddev>1.0</stddev>
+				</noise>
+			</camera>
+			<plugin name="ensenso_plugin" filename="libgazebo_ros_openni_kinect.so">
+				<baseline>0.1</baseline>
+				<alwaysOn>true</alwaysOn>
+				<!-- Keep this zero, update_rate in the parent <sensor> tag
+				will control the frame rate. -->
+				<updateRate>0.0</updateRate>
+				<cameraName>${name}</cameraName>
+				<imageTopicName>/${name}/image_raw</imageTopicName>
+				<cameraInfoTopicName>/${name}/camera_info</cameraInfoTopicName>
+				<depthImageTopicName>/${name}/image_raw</depthImageTopicName>
+				<depthImageInfoTopicName>/${name}/camera_info</depthImageInfoTopicName>
+				<pointCloudTopicName>/${name}/ensenso_cloud</pointCloudTopicName>
+				<frameName>${name}_body</frameName>
+				<pointCloudCutoff>${focus_length - 0.5}</pointCloudCutoff>
+				<pointCloudCutoffMax>${focus_length + 0.5}</pointCloudCutoffMax>
+			</plugin>
+			<always_on>true</always_on>
+			<update_rate>1.0</update_rate>
+		</sensor>
+	</gazebo>
+</xacro:macro>
 </robot>
